Commit message: fix map path

File: maps/tue_hallway_RLtoAL/map.urdf (robot description, URDF)
Before this commit: robot map, 1 links, 0 joints
Links:
- link map: geometry collision mesh filename=package://ropod_sim_model/maps/tue_hallway_RLtoAL/map.stl scale=0.001 0.001 0.003; visual mesh filename=package://ropod_sim_model/maps/tue_hallway_RLtoAL/map.stl scale=0.001 0.001 0.003

Commit message: Add file to test heighmaps

File: maps/tue_hallway_RLtoAL/map.urdf (robot description, URDF)
Before this commit: robot map, 1 links, 0 joints
Links:
- link map: mass 10000 -> None; geometry collision heightmap ; visual heightmap 
